Commit message: Added collision tags to the urdf model.

File: urdf/myrobot.urdf (robot description, URDF)
Before this commit: robot basic_robot, 5 links, 4 joints
Links:
- link base_link: geometry collision box size=1.0 1.0 0.1; visual box size=1.0 1.0 0.1
- link left_back_wheel: geometry collision cylinder length=0.1 radius=0.1; visual cylinder length=0.1 radius=0.1
- link left_front_wheel: geometry collision cylinder length=0.1 radius=0.1; visual cylinder length=0.1 radius=0.1
- link right_back_wheel: geometry collision cylinder length=0.1 radius=0.1; visual cylinder length=0.1 radius=0.1
- link right_front_wheel: geometry collision cylinder length=0.1 radius=0.1; visual cylinder length=0.1 radius=0.1

Commit message: Added interia tags to URDF model. Used ROS wiki.

File: urdf/myrobot.urdf (robot description, URDF)
Before this commit: robot basic_robot, 5 links, 4 joints
Links:
- link base_link: mass None -> 10
- link left_back_wheel: mass None -> 1
- link left_front_wheel: mass None -> 1
- link right_back_wheel: mass None -> 1
- link right_front_wheel: mass None -> 1
