Commit message: Fixed syntax errors.

File: urdf/myrobot.xacro (robot description, xacro)
@@ -42,5 +42,5 @@
 <link name="base_link">
     <visual>
-    <origin xyz=${base_origin}/>
+    <origin xyz="${base_origin}"/>
       <geometry>
          <box size="${length} ${width} ${height}"/>
@@ -48,5 +48,5 @@
     </visual>
     <collision>
-      <origin xyz=${base_origin}/>
+      <origin xyz="${base_origin}"/>
       <geometry>
          <box size="${length} ${width} ${height}"/>
@@ -103,5 +103,5 @@
       <origin rpy="${wheel_origin_rpy}" />
       <geometry>
-        <cylinder length=${wheel_len}" radius="${wheel_radius}"/>
+        <cylinder length="${wheel_len}" radius="${wheel_radius}"/>
       </geometry>
       <material name="blue"/>
@@ -110,5 +110,5 @@
       <origin rpy="${wheel_origin_rpy}" />
       <geometry>
-        <cylinder length=${wheel_len}" radius="${wheel_radius}"/>
+        <cylinder length="${wheel_len}" radius="${wheel_radius}"/>
       </geometry>
     </collision>

Commit message: Fixed base link URDF inertia warning.

File: urdf/myrobot.xacro (robot description, xacro)
@@ -40,4 +40,11 @@
 <!--xacro macro for left_back_wheel_joint-->
 <xacro:property name="left_back_wheel_joint_xyz" value="-0.4 -0.5 0.1" />
+<!-- Dummy link to get rid of  base_link has an inertia specified in the URDF error -->
+<link name="dummy"/>
+<!-- Dummy joint to get rid of  base_link has an inertia specified in the URDF error -->
+<joint name="dummy_joint" type="fixed">
+  <parent link="dummy" />
+  <child link="base_link" />
+</joint>
 <link name="base_link">
     <visual>

File: urdf/myrobot1.0.urdf (robot description, URDF)
Before this commit: robot basic_robot, 5 links, 4 joints
Links:
- added link dummy
Joints:
- added joint dummy_joint: type fixed, parent dummy, child base_link

Commit message: In process of creating wheel macros.

File: urdf/myrobot.xacro (robot description, xacro)
@@ -151,4 +151,40 @@
     <origin rpy="0 0 0" xyz="${left_back_wheel_joint_xyz}"/>
   </joint>
+  <!-- create a xacro macro for the wheels links -->
+  <xacro:macro name="wheel" params="prefix suffix reflect">
+      <link name="${prefix}_${suffix}_wheel">
+          <visual>
+            <origin xyz="0 0 0" rpy="${pi/2} 0 0" />
+            <geometry>
+              <cylinder radius="${wheel_radius}" length="${wheel_len}"/>
+            </geometry>
+            <material name="black"/>
+          </visual>
+          <collision>
+            <origin xyz="0 0 0" rpy="${pi/2} 0 0" />
+            <geometry>
+              <cylinder radius="${wheel_radius}" length="${wheel_len}"/>
+            </geometry>
+          </collision>
+          <xacro:wheel_inertia mass="1"/>
+      </link>
+      <!-- create xacro macro fo wheel joint -->
+      <joint name="${prefix}_${suffix}_wheel_joint" type="continuous">
+          <axis xyz="${wheel_axis}" rpy="0 0 0" />
+          <parent link="${prefix}_base"/>
+          <child link="${prefix}_${suffix}_wheel"/>
+          <origin xyz="${baselen*reflect/3} 0 -${wheeldiam/2+.05}" rpy="0 0 0"/>
+      </joint>
+  </xacro:macro>
+<!--wheel/joint_0 code inspired from -->
+<!-- https://github.com/ZBO-R8io/Roberto/blob/main/backups/lunarbot/urdf/lunarbot.xacro -->
+<!-- change these values -->
+  <xacro:wheel suffix="0" reflect_x="1" reflect_y="1" reflect_z="-1" />
+  <!--wheel/joint_1-->
+  <xacro:wheel suffix="1" reflect_x="1" reflect_y="-1" reflect_z="-1" />
+  <!--wheel/joint_2-->
+  <xacro:wheel suffix="2" reflect_x="-1" reflect_y="1" reflect_z="-1" />
+  <!--wheel/joint_3-->
+  <xacro:wheel suffix="3" reflect_x="-1" reflect_y="-1" reflect_z="-1" />
   <!-- Gazebo plugin for ROS Control -->
   <gazebo>

Commit message: Added wheel macros.

File: urdf/myrobot.xacro (robot description, xacro)
@@ -62,95 +62,6 @@
     <xacro:base_inertial mass="10"/>
 </link>
-<link name="right_front_wheel">
-    <visual>
-      <origin rpy="${wheel_origin_rpy}"/>
-      <geometry>
-        <cylinder length="${wheel_len}" radius="${wheel_radius}"/>
-      </geometry>
-      <material name="blue"/>
-    </visual>
-    <collision>
-      <origin rpy="${wheel_origin_rpy}"/>
-      <geometry>
-         <cylinder length="${wheel_len}" radius="${wheel_radius}"/>
-      </geometry>
-    </collision>
-    <xacro:wheel_inertia mass="1"/>
-</link>
-<joint name="right_front_wheel_joint" type="continuous">
-    <parent link="base_link" />
-    <child link="right_front_wheel" />
-    <axis xyz="${wheel_axis}"/>
-    <origin rpy="0 0 0 " xyz="${right_front_wheel_joint_xyz}"/>
-</joint>
-<link name="left_front_wheel">
-    <visual>
-      <origin rpy="${wheel_origin_rpy}"/>
-      <geometry>
-        <cylinder length="${wheel_len}" radius="${wheel_radius}"/>
-      </geometry>
-      <material name="blue"/>
-    </visual>
-    <collision>
-      <origin rpy="${wheel_origin_rpy}"/>
-      <geometry>
-        <cylinder length="${wheel_len}" radius="${wheel_radius}"/>
-      </geometry>
-    </collision>
-    <xacro:wheel_inertia mass="1"/>
-</link>
-<joint name="left_front_wheel_joint" type="continuous">
-    <parent link="base_link" />
-    <child link="left_front_wheel" />
-    <axis xyz="${wheel_axis}"/>
-    <origin rpy="0 0 0" xyz="${left_front_wheel_joint_xyz}"/>
-</joint>
-<link name="right_back_wheel">
-    <visual>
-      <origin rpy="${wheel_origin_rpy}" />
-      <geometry>
-        <cylinder length="${wheel_len}" radius="${wheel_radius}"/>
-      </geometry>
-      <material name="blue"/>
-    </visual>
-    <collision>
-      <origin rpy="${wheel_origin_rpy}" />
-      <geometry>
-        <cylinder length="${wheel_len}" radius="${wheel_radius}"/>
-      </geometry>
-    </collision>
-    <xacro:wheel_inertia mass="1"/>
-</link>
-<joint name="right_back_wheel_joint" type="continuous">
-    <parent link="base_link" />
-    <child link="right_back_wheel" />
-    <axis xyz="${wheel_axis}"/>
-    <origin rpy="0 0 0" xyz="${right_back_wheel_joint_xyz}"/>
-</joint>
-<link name="left_back_wheel">
-    <visual>
-      <origin rpy="${wheel_origin_rpy}"/>
-      <geometry>
-        <cylinder length="${wheel_len}" radius="${wheel_radius}"/>
-      </geometry>
-      <material name="blue"/>
-    </visual>
-    <collision>
-      <origin rpy="${wheel_origin_rpy}"/>
-      <geometry>
-        <cylinder length="${wheel_len}" radius="${wheel_radius}"/>
-      </geometry>
-    </collision>
-    <xacro:wheel_inertia mass="1"/>
-</link>
-<joint name="left_back_wheel_joint" type="continuous">
-    <parent link="base_link" />
-    <child link="left_back_wheel" />
-    <!-- axis on which it will move -->
-    <axis xyz="${wheel_axis}"/>
-    <origin rpy="0 0 0" xyz="${left_back_wheel_joint_xyz}"/>
-  </joint>
   <!-- create a xacro macro for the wheels links -->
-  <xacro:macro name="wheel" params="prefix suffix reflect">
+  <xacro:macro name="wheel" params="prefix suffix reflect_x reflect_y reflect_z">
       <link name="${prefix}_${suffix}_wheel">
           <visual>
@@ -172,7 +83,7 @@
       <joint name="${prefix}_${suffix}_wheel_joint" type="continuous">
           <axis xyz="${wheel_axis}" rpy="0 0 0" />
-          <parent link="${prefix}_base"/>
+          <parent link="base_link"/>
           <child link="${prefix}_${suffix}_wheel"/>
-          <origin xyz="${baselen*reflect/3} 0 -${wheeldiam/2+.05}" rpy="0 0 0"/>
+          <origin xyz="${reflect_x * 0.4} ${reflect_y * 0.5} ${reflect_z * 0.1}" rpy="0 0 0"/>
       </joint>
   </xacro:macro>
@@ -180,11 +91,11 @@
 <!-- https://github.com/ZBO-R8io/Roberto/blob/main/backups/lunarbot/urdf/lunarbot.xacro -->
 <!-- change these values -->
-  <xacro:wheel suffix="0" reflect_x="1" reflect_y="1" reflect_z="-1" />
+  <xacro:wheel prefix="right" suffix="0" reflect_x="1" reflect_y="1" reflect_z="1" />
   <!--wheel/joint_1-->
-  <xacro:wheel suffix="1" reflect_x="1" reflect_y="-1" reflect_z="-1" />
+  <xacro:wheel prefix="left" suffix="1" reflect_x="1" reflect_y="-1" reflect_z="1" />
   <!--wheel/joint_2-->
-  <xacro:wheel suffix="2" reflect_x="-1" reflect_y="1" reflect_z="-1" />
+  <xacro:wheel prefix="right" suffix="2" reflect_x="-1" reflect_y="1" reflect_z="1" />
   <!--wheel/joint_3-->
-  <xacro:wheel suffix="3" reflect_x="-1" reflect_y="-1" reflect_z="-1" />
+  <xacro:wheel prefix="left" suffix="3" reflect_x="-1" reflect_y="-1" reflect_z="1" />
   <!-- Gazebo plugin for ROS Control -->
   <gazebo>

Commit message: Edited xacro file

File: urdf/myrobot.xacro (robot description, xacro)
@@ -49,5 +49,5 @@
 <link name="base_link">
     <visual>
-    <origin xyz="${base_origin}"/>
+    <!-- <origin xyz="${base_origin}"/> -->
       <geometry>
          <box size="${length} ${width} ${height}"/>
@@ -55,5 +55,5 @@
     </visual>
     <collision>
-      <origin xyz="${base_origin}"/>
+      <!-- <origin xyz="${base_origin}"/> -->
       <geometry>
          <box size="${length} ${width} ${height}"/>
@@ -85,6 +85,26 @@
           <parent link="base_link"/>
           <child link="${prefix}_${suffix}_wheel"/>
-          <origin xyz="${reflect_x * 0.4} ${reflect_y * 0.5} ${reflect_z * 0.1}" rpy="0 0 0"/>
+          <origin xyz="${reflect_x * 0.4} ${reflect_y * 0.5} ${reflect_z * 0.05}" rpy="0 0 0"/>
       </joint>
+      <!-- This block provides the simulator (Gazebo) with information on a few additional
+      physical properties. See http://gazebosim.org/tutorials/?tut=ros_urdf for more-->
+      <gazebo reference="${prefix}_${suffix}_wheel">
+        <mu1 value="200.0"/>
+        <mu2 value="100.0"/>
+        <kp value="10000000.0" />
+        <kd value="1.0" />
+        <material>Gazebo/Grey</material>
+      </gazebo>
+      <!-- This block connects the wheel joint to an actuator (motor), which informs both
+          simulation and visualization of the robot -->
+      <transmission name="${prefix}_${suffix}_wheel_trans">
+        <type>transmission_interface/SimpleTransmission</type>
+        <actuator name="${prefix}_${suffix}_wheel_motor">
+          <mechanicalReduction>1</mechanicalReduction>
+        </actuator>
+        <joint name="${prefix}_${suffix}_wheel_joint">
+          <hardwareInterface>hardware_interface/VelocityJointInterface</hardwareInterface>
+        </joint>
+      </transmission>
   </xacro:macro>
 <!--wheel/joint_0 code inspired from -->
