Commit message: Changed file locations in file.

File: urdf/nasa_bot.xacro (robot description, xacro)
@@ -32,5 +32,5 @@
       <visual>
         <geometry>
-          <mesh filename="package://lunarbot/meshes/base_link2.stl"/>
+          <mesh filename="package://new_robot_urdf/meshes/base_link2.stl"/>
         </geometry>
         <material name="${body_color}"/>
@@ -218,5 +218,5 @@
         <origin xyz="${auger_link_origin}"/>
         <geometry>
-           <mesh filename="package://lunarbot/meshes/auger.stl"/>
+           <mesh filename="package://new_robot_urdf/meshes/auger.stl"/>
         </geometry>
         <material name="${auger_color}"/>
@@ -261,5 +261,5 @@
   <gazebo>
 	  <plugin name="gazebo_ros_control" filename="libgazebo_ros_control.so"/>
-	  <robotNamespace>/lunarbot</robotNamespace>
+	  <robotNamespace>/new_robot_urdf</robotNamespace>
 	</gazebo>
 </robot>
